File: PCB/Inverter.kicad_sch (KiCad schematic)
At the start: 87 parts, among them J1 Conn_01x02, J2 Conn_01x05_Pin, J3 Conn_01x05_Pin, Q1 STP110N8F6, Q2 STP110N8F6, Q3 STP110N8F6, Q4 STP110N8F6, Q5 STP110N8F6, Q6 STP110N8F6, U1 XL7015, U10 L7805, U2 MountingHole_Pad, U3 ACS712-20A, U4 ACS712-20A, U5 ACS712-20A, U6 IR2104, U7 IR2104, U8 IR2104

Commit message: Change#004
Add new schematics files
Parts:
- removed U6, U7, U8: IR2104, Package_SO:SOIC-8_3.9x4.9mm_P1.27mm, symbol Driver_FET:IR2104
- added C25, C27, C28, C29: 100nF, Capacitor_SMD:C_0805_2012Metric_Pad1.18x1.45mm_HandSolder, symbol Device:C
- added C26: 10uF, Capacitor_SMD:C_0805_2012Metric_Pad1.18x1.45mm_HandSolder, symbol Device:C
- added R19: 1K, Resistor_SMD:R_0805_2012Metric_Pad1.20x1.40mm_HandSolder, symbol Device:R_US
- added U6, U7, U8: IR2101, Package_SO:SOIC-8_3.9x4.9mm_P1.27mm, symbol Driver_FET:IR2101
- added U9: AMS1117-3.3, Package_TO_SOT_SMD:SOT-223-3_TabPin2, symbol Regulator_Linear:AMS1117-3.3
- C24: value 1000uF 16V -> 1000uF 6.3V
- R12: value 10K -> 100K
- R2: value 10K -> 7K5
- R5, R6, R7: value 1K -> 10K
Connections:
- net +10V: now also U6.1 (VCC), U7.1 (VCC), U8.1 (VCC)
- net +5V: now also C25.1, U9.3 (VI)
- net GND: now also U3.3 (IP-), U3.4 (IP-), U4.3 (IP-), U4.4 (IP-), U5.3 (IP-), U5.4 (IP-), C25.2, C26.1, C27.2, C28.2, C29.1, U6.4 (COM), U7.4 (COM), U8.4 (COM), U9.1 (GND); no longer D16.2 (A), D18.2 (A), D20.2 (A), Q2.3 (S), Q4.3 (S), Q6.3 (S)
- net at D12.1 (K), R16.2: now also U7.5 (LO)
- net at C16.2, D6.1 (K): now also U6.8 (VB)
- net at D11.1 (K), R15.2: now also U7.7 (HO)
- net at C17.2, D7.1 (K): now also U7.8 (VB)
- net at D14.1 (K), R18.2: now also U8.5 (LO)
- net at D13.1 (K), R17.2: now also U8.7 (HO)
- net at C18.2, D8.1 (K): now also U8.8 (VB)
- net at D10.1 (K), R14.2: now also U6.5 (LO)
- net at D9.1 (K), R13.2: now also U6.7 (HO)
- net +5V_Fuse renamed +3.3V
- net +3.3V: now also C26.2, C27.1, R19.2, U9.2 (VO); no longer F1.1, J2.5 (Pin_5), J3.5 (Pin_5)
- net U_IN renamed U_POW
- net U_POW: now also U2.1, U6.6 (VS); no longer U3.3 (IP-), U3.4 (IP-)
- net U_OUT renamed U_SENS
- net U_SENS: now also D16.2 (A), Q2.3 (S); no longer U2.1
- net V_IN renamed V_POW
- net V_POW: now also V1.1, U7.6 (VS); no longer U4.3 (IP-), U4.4 (IP-)
- net V_OUT renamed V_SENS
- net V_SENS: now also D18.2 (A), Q4.3 (S); no longer V1.1
- net W_IN renamed W_POW
- net W_POW: now also W1.1, U8.6 (VS); no longer U5.3 (IP-), U5.4 (IP-)
- net W_OUT renamed W_SENS
- net W_SENS: now also D20.2 (A), Q6.3 (S); no longer W1.1
- new net: C29.2, J2.5 (Pin_5), R19.1
- new net: C28.1, F1.1, J3.5 (Pin_5)
- new net H_PWM_U: U6.2 (HIN)
- new net H_PWM_V: U7.2 (HIN)
- new net H_PWM_W: U8.2 (HIN)
- new net L_PWM_U: U6.3 (LIN)
- new net L_PWM_V: U7.3 (LIN)
- new net L_PWM_W: U8.3 (LIN)
Other:
- moved on the sheet: C1, C10, C11, C12, C13, C14, C15, C16, C17, C18, C19, C20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
