File: PCB/Inverter.kicad_sch (KiCad schematic)
At the start: 94 parts, among them J1 Conn_01x02, J2 Conn_01x05_Pin, J3 Conn_01x05_Pin, Q1 STP110N8F6, Q2 STP110N8F6, Q3 STP110N8F6, Q4 STP110N8F6, Q5 STP110N8F6, Q6 STP110N8F6, U1 XL7015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

Commit message: Change#006
Updated the description - changed the power rating from 650 to 1000 W.
Parts:
- added R20: 100K, Resistor_SMD:R_0805_2012Metric_Pad1.20x1.40mm_HandSolder, symbol Device:R_US
- R19: value 1K -> 10
- R2: value 7K5 -> 10K
Connections:
- net CWR: now also J2.2 (Pin_2); no longer J2.3 (Pin_3)
- net GND: no longer J2.2 (Pin_2)
- net POT: now also J2.3 (Pin_3); no longer J2.4 (Pin_4)
- net at C29.2, J2.5 (Pin_5), R19.1: now also J2.4 (Pin_4)
- net at C1.1, D1.1 (K), U1.1 (Vin): now also R20.2; no longer R1.1
- new net: R1.1, R20.1
Other:
- moved on the sheet: C1, C10, C11, C12, C13, C14, C15, C16, C17, C18, C19, C20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
